File: minimal_max32650/minimal_max32650.kicad_sch (KiCad schematic)
At the start: 38 parts, among them J1 FTSH-105-01-L-DV-K, U1 MAX32650GCE+, U2 ADP225ACPZ-R7

Commit message: development backup
Parts:
- added C28: 4.7 µF, capacitor_footprints:C_0603_1608Metric, symbol UNITED_CAPACITORS_DATA_BASE:C_C1608X7S1A475K080AC
- added C29: 0.1uF, capacitor_footprints:C_0402_1005Metric, symbol UNITED_CAPACITORS_DATA_BASE:C_GCM155R71H104KE02D
- added C30: 1 µF, capacitor_footprints:C_0402_1005Metric, symbol UNITED_CAPACITORS_DATA_BASE:C_C1005X6S1C105K050BC
- added TP5, TP6: TestPoint, test_point_footprints:TestPoint_THTPad_Castelated, symbol UNITED_TEST_POINTS:TestPoint_Castelated
- added U3: MAXQ1065GTC+, analog_devices_footprints:21-0664_TD1233&plus_1C_MXM, symbol UNITED_IC_ADI:U_MAXQ1065GTC+
- renumbered C26 to C24, C24 to C25, C25 to C26, R2 to R1, R4 to R2, R1 to R3, R3 to R4, TP4 to TP3, TP3 to TP4
Connections:
- net 3V3: now also C28.1, C29.1, TP5.1, U3.12 (VDD)
- net GND: now also C28.2, C29.2, C30.2, TP6.1, U3.13 (EP), U3.6 (GND)
- net MAXQ1065_RDY: now reaches U1.1 (P2.16)
- net MAXQ1065_RDY: now also U3.11 (RDY)
- net SPI0_SS0: now reaches U1.10 (P0.22)
- net SPI0_SS0: now also U3.5 (SPIS_SS)
- net SPI0_MISO: now reaches U1.138 (P3.1)
- net SPI0_MISO: now also U3.4 (SPIS_MISO)
- net SPI0_MOSI: now reaches U1.141 (P3.2)
- net SPI0_MOSI: now also U3.3 (SPIS_MOSI)
- net SPI0_SCK: now reaches U1.142 (P3.3)
- net SPI0_SCK: now also U3.2 (SPIS_SCK)
- net MAXQ1065_WDI: now reaches U1.2 (P0.1)
- net MAXQ1065_WDI: now also U3.9 (WDI)
- net MAXQ1065_PDWN: now reaches U1.3 (P0.2)
- net MAXQ1065_PDWN: now also U3.7 (PDWN)
- new net: C30.1, U3.1 (CEXT)
- no-connect marks 1 -> 3
Other:
- moved on the sheet: C24, C25, C26, C9, R1, R2, R3, R4, TP1, TP2, TP3, TP4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

Commit message: development backup
Parts:
- added C5: 0.1uF, capacitor_footprints:C_0402_1005Metric, symbol UNITED_CAPACITORS_DATA_BASE:C_GCM155R71H104KE02D
- added D1, D2: 1.8 V, diode_footprints:LED_GREEN_0402_1005Metric, symbol UNITED_DIODES_DATA_BASE:D_APHHS1005CGCK
- added Q1, Q2: 50 V, transistor_footprints:SOT23-3, symbol UNITED_TRANSISTORS_DATA_BASE:Q_BSS138-7-F
- added R1, R2, R3: 10k, resistor_footprints:R_0402_1005Metric, symbol UNITED_RESISTORS_DATA_BASE:R_ERJ-2RKF1002X
- added R4, R5: 1 kΩ, resistor_footprints:R_0402_1005Metric, symbol UNITED_RESISTORS_DATA_BASE:R_ERJ-2RKF1001X
- added U1: ADT75BRMZ, analog_devices_footprints:RM_8_ADI, symbol UNITED_IC_ADI:U_ADT75BRMZ
- renumbered C9 to C10, C10 to C11, C11 to C12, C12 to C13, C13 to C14, C14 to C15, C15 to C16, C16 to C17, C17 to C18, C18 to C19, C30 to C20, C19 to C21, C20 to C22, C21 to C23, C22 to C24, C23 to C25, C28 to C26, C29 to C27, C27 to C28, C25 to C29, C24 to C30, C26 to C31, C5 to C6, C6 to C7, C7 to C8, C8 to C9, R2 to R6, R4 to R7, R1 to R8, R3 to R9, TP2 to TP1, TP4 to TP2, TP1 to TP3, TP3 to TP4, TP6 to TP5, TP5 to TP6, U1 to U2, U2 to U4
Connections:
- net 3V3: now also C5.1, R1.1, R2.1, R3.1, R4.1, R5.1, U1.8 (VDD)
- net GND: now also C5.2, Q1.2 (S), Q2.2 (S), U1.4 (GND), U1.5 (A2), U1.6 (A1), U1.7 (A0)
- net LED2: now reaches U2.143 (P2.14)
- net LED2: now also Q1.1 (G)
- net LED1: now reaches U2.144 (P2.15)
- net LED1: now also Q2.1 (G)
- net I2C1_SDA: now reaches U2.19 (P2.17)
- net I2C1_SDA: now also R3.2, U1.1 (SDA)
- net I2C1_SCL: now reaches U2.20 (P2.18)
- net I2C1_SCL: now also R2.2, U1.2 (SCL)
- net ADT75_OS/ALERT: now reaches U2.39 (P1.1)
- net ADT75_OS/ALERT: now also R1.2, U1.3 (OS/ALERT)
- new net: D2.1, Q2.3 (D)
- new net: D2.2, R5.2
- new net: D1.2, R4.2
- new net: D1.1, Q1.3 (D)
- no-connect marks 3 -> 27
Other:
- moved on the sheet: C28, J1

Commit message: Add SPI interface color mappings to KiCad project
Parts:
- added C2: 100 nF, capacitor_footprints:C_0402_1005Metric, symbol UNITED_CAPACITORS_DATA_BASE:C_GCM155R71H104KE02D
- added U2: MX25U6432FZNI02, macronix_footprints:WSON-8_6X5_MAC, symbol UNITED_IC_MACRONIX:U_MX25U6432FZNI02
- C1: renamed from C5; value 0.1uF -> 100 nF; 3dviewer Link (none) -> https://3dviewer.net/index.html#model=https://github.com/io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; Capacitor Type (none) -> Ceramic
- C28: renamed from C27; value 0.1uF -> 100 nF; 3dviewer Link (none) -> https://3dviewer.net/index.html#model=https://github.com/io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; Capacitor Type (none) -> Ceramic
- C29: renamed from C28; value 0.1uF -> 100 nF; 3dviewer Link (none) -> https://3dviewer.net/index.html#model=https://github.com/io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; Capacitor Type (none) -> Ceramic
- renumbered C9 to C10, C10 to C11, C11 to C12, C12 to C13, C13 to C14, C14 to C15, C15 to C16, C16 to C17, C17 to C18, C18 to C19, C19 to C20, C20 to C21, C21 to C22, C22 to C23, C23 to C24, C24 to C25, C25 to C26, C26 to C27, C1 to C3, C29 to C30, C30 to C31, C31 to C32, C2 to C4, C3 to C5, C4 to C6, C6 to C7, C7 to C8, C8 to C9, U2 to U3, U3 to U4, U4 to U5
Connections:
- net 1V8: now also C2.1, U2.8 (VCC)
- net GND: now also C2.2, U2.4 (GND), U2.9 (GND)
- net SPIXF_SS0: now reaches U3.12 (P0.7)
- net SPIXF_SS0: now also U2.1 (~{CS})
- net SPIXF_SCK: now reaches U3.13 (P0.8)
- net SPIXF_SCK: now also U2.6 (SCLK)
- net SPIXF_SDIO1: now reaches U3.15 (P0.9)
- net SPIXF_SDIO1: now also U2.2 (SO/SIO1)
- net SPIXF_SDIO0: now reaches U3.17 (P0.10)
- net SPIXF_SDIO0: now also U2.5 (SI/SIO0)
- net SPIXF_SDIO2: now reaches U3.22 (P0.11)
- net SPIXF_SDIO2: now also U2.3 (~{WP}/SIO2)
- net SPIXF_SDIO3: now reaches U3.23 (P0.12)
- net SPIXF_SDIO3: now also U2.7 (~{RESET}/SIO3)
Other:
- moved on the sheet: C30, C31, C32, R6, R7, R8, R9, TP1, TP2, TP3, TP4, TP5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

Commit message: development backup
Parts:
- added C35, C36, C39, C40: 100 nF, capacitor_footprints:C_0402_1005Metric, symbol UNITED_CAPACITORS_DATA_BASE:C_GCM155R71H104KE02D
- added C37, C38: 1 µF, capacitor_footprints:C_0402_1005Metric, symbol UNITED_CAPACITORS_DATA_BASE:C_C1005X6S1C105K050BC
- added U6: S80KS5122GABHM020, infineon_footprints:PG-BGA-24-801, symbol UNITED_IC_INFINEON:U_S80KS5122GABHM020
Connections:
- net 1V8: now also C35.1, C36.1, C37.1, C38.1, C39.1, C40.1, U6.B4 (VCC), U6.D1 (VCCQ), U6.E4 (VCCQ)
- net GND: now also C35.2, C36.2, C37.2, C38.2, C39.2, C40.2, U6.B3 (VSS), U6.C1 (VSSQ), U6.E5 (VSSQ)
- net CS1__P3.0: now reaches U3.44 (P3.0)
- net RESET__P1.10: now reaches U3.50 (P1.10)
- net RESET__P1.10: now also U6.A4 (~{RESET})
- net CS0__P1.11: now reaches U3.52 (P1.11)
- net CS0__P1.11: now also U6.A3 (~{CS})
- net D0__P1.12: now reaches U3.53 (P1.12)
- net D0__P1.12: now also U6.D3 (DQ0)
- net D4__P1.13: now reaches U3.56 (P1.13)
- net D4__P1.13: now also U6.D5 (DQ4)
- net D1__P1.15: now reaches U3.58 (P1.15)
- net D1__P1.15: now also U6.D2 (DQ1)
- net D5__P1.16: now reaches U3.59 (P1.16)
- net D5__P1.16: now also U6.E3 (DQ5)
- net D2__P1.19: now reaches U3.62 (P1.19)
- net D2__P1.19: now also U6.C4 (DQ2)
- net D6__P1.18: now reaches U3.63 (P1.18)
- net D6__P1.18: now also U6.E2 (DQ6)
- net CLK_N: now reaches U3.64 (~{HYP_CLK})
- net CLK_N: now also U6.B1 (~{CK})
- net CLK_P: now reaches U3.65 (HYP_CLK)
- net CLK_P: now also U6.B2 (CK)
- net D3__P1.20: now reaches U3.66 (P1.20)
- net D3__P1.20: now also U6.D4 (DQ3)
- net D7__P1.21: now reaches U3.67 (P1.21)
- net D7__P1.21: now also U6.E1 (DQ7)
- net RWDS__P1.14: now reaches U3.68 (P1.14)
- net RWDS__P1.14: now also U6.C3 (RWDS)

Commit message: development backup
Parts:
- renumbered C40 to C1, C4 to C10, C5 to C11, C6 to C12, C7 to C13, C8 to C14, C9 to C15, C10 to C16, C11 to C17, C12 to C18, C13 to C19, C39 to C2, C14 to C20, C15 to C21, C16 to C22, C17 to C23, C18 to C24, C19 to C25, C20 to C26, C21 to C27, C22 to C28, C23 to C29, C38 to C3, C24 to C30, C25 to C31, C26 to C32, C27 to C33, C28 to C34, C31 to C35, C30 to C36, C32 to C37, C29 to C38, C35 to C4, C1 to C5, C36 to C6, C37 to C7, C2 to C8, C3 to C9, R8 to R4, R6 to R5, R4 to R6, R9 to R7, R7 to R8, R5 to R9, TP3 to TP1, TP1 to TP2, TP4 to TP3, TP2 to TP4, TP6 to TP5, TP5 to TP6, U6 to U2, U2 to U3, U3 to U4, U4 to U5, U5 to U6

Commit message: development backup
Parts:
- added TP1, TP2, TP3, TP4, TP5: TestPoint, test_point_footprints:TestPoint_THTPad_Castelated, symbol UNITED_TEST_POINTS:TestPoint_Castelated
- renumbered C36 to C35, C35 to C36, R5 to R4, R8 to R5, R4 to R6, R6 to R8, TP5 to TP10, TP6 to TP11, TP2 to TP6, TP4 to TP7, TP1 to TP8, TP3 to TP9
Connections:
- net at U4.30 (P0.16): now also TP5.1
- net at U4.31 (P0.17): now also TP4.1
- net at U4.32 (P0.18): now also TP3.1
- net at U4.35 (P0.20): now also TP2.1
- net at U4.36 (P0.21): now also TP1.1
- no-connect marks 27 -> 33

Commit message: development backup
Parts:
- added TP1, TP14, TP15, TP16, TP2, TP3, TP4, TP5, TP6, TP7, TP8: TestPoint, test_point_footprints:TestPoint_THTPad_Castelated, symbol UNITED_TEST_POINTS:TestPoint_Castelated
- renumbered TP2 to TP10, TP3 to TP11, TP4 to TP12, TP5 to TP13, TP6 to TP17, TP7 to TP18, TP8 to TP19, TP9 to TP20, TP10 to TP21, TP11 to TP22, TP1 to TP9
Connections:
- net at U4.100 (P0.27): now also TP15.1
- net at U4.103 (P0.26): now also TP16.1
- net at U4.45 (P1.4): now also TP7.1
- net at U4.46 (P1.8): now also TP6.1
- net at U4.48 (P1.9): now also TP5.1
- net at U4.49 (P1.6): now also TP4.1
- net at U4.70 (P1.23): now also TP3.1
- net at U4.71 (P1.30): now also TP2.1
- net at U4.72 (P1.25): now also TP1.1
- net at U4.75 (P1.22): now also TP8.1
- net at U4.90 (P3.9): now also TP14.1

Commit message: development backup
Parts:
- added TP14, TP15, TP16, TP17, TP20, TP21, TP22, TP23, TP24, TP25, TP26, TP28, TP29, TP30, TP31, TP32, TP33, TP34, TP35, TP36, TP37, TP38, TP39: TestPoint, test_point_footprints:TestPoint_THTPad_Castelated, symbol UNITED_TEST_POINTS:TestPoint_Castelated
- renumbered R8 to R6, R6 to R7, R7 to R8, TP15 to TP18, TP14 to TP19, TP16 to TP27, TP17 to TP40, TP18 to TP41, TP19 to TP42, TP20 to TP43, TP21 to TP44, TP22 to TP45
Connections:
- net at U4.115 (P1.26): now also TP32.1
- net at U4.116 (P1.27): now also TP39.1
- net at U4.117 (P1.28): now also TP31.1
- net at U4.118 (P1.29): now also TP38.1
- net at U4.120 (P2.0): now also TP37.1
- net at U4.121 (P2.1): now also TP30.1
- net at U4.122 (P2.2): now also TP36.1
- net at U4.123 (P2.3): now also TP29.1
- net at U4.124 (P2.4): now also TP35.1
- net at U4.125 (P2.5): now also TP28.1
- net at U4.127 (P2.6): now also TP26.1
- net at U4.129 (P2.7): now also TP25.1
- net at U4.130 (P2.8): now also TP34.1
- net at U4.131 (P2.9): now also TP24.1
- net at U4.133 (P2.25): now also TP23.1
- net at U4.134 (P2.10): now also TP33.1
- net at U4.91 (P3.6): now also TP14.1
- net at U4.92 (P1.24): now also TP20.1
- net at U4.93 (P1.31): now also TP15.1
- net at U4.94 (P3.8): now also TP21.1
- net at U4.95 (P3.5): now also TP16.1
- net at U4.96 (P3.7): now also TP17.1
- net at U4.97 (P3.4): now also TP22.1
- no-connect marks 33 -> 35
