File: minimal_max32650/minimal_max32650.kicad_sch (KiCad schematic)
At the start: 103 parts, among them J1 FTSH-105-01-L-DV-K, Q1 50 V, Q2 50 V, U1 ADT75BRMZ, U2 S80KS5122GABHM020, U3 MX25U6432FZNI02, U4 MAX32650GCE+, U5 MAXQ1065GTC+, U6 ADP225ACPZ-R7

Commit message: development backup
Parts:
- added J1: CLP-150-02-G-D-BE, connector_footprints:CLP-141-02-G-D-BE, symbol UNITED_CONNECTORS_DATA_BASE:J_CLP-141-02-G-D-BE
- added MB1: mouse-bite-midle-50mil-200mil, mouse_bite_footprints:mouse-bite-50mil-2138mil, symbol UNITED_MOUSE_BITES_DATA_BASE:mouse-bite-50mil-2138mil
- renumbered D2 to D1, D1 to D2, J1 to J2, Q2 to Q1, Q1 to Q2, R7 to R6, R8 to R7, R9 to R8, R6 to R9, TP40 to TP38, TP41 to TP39, TP5 to TP4, TP38 to TP40, TP39 to TP41, TP45 to TP44, TP44 to TP45, TP6 to TP5, TP7 to TP6, TP4 to TP7
Connections:
- net 3V3: now also J1.81
- net GND: now also J1.10, J1.12, J1.14, J1.16, J1.18, J1.2, J1.20, J1.22, J1.24, J1.26, J1.28, J1.30, J1.32, J1.34, J1.36, J1.38, J1.4, J1.40, J1.42, J1.44, J1.46, J1.48, J1.50, J1.52, J1.54, J1.56, J1.58, J1.6, J1.60, J1.62, J1.64, J1.66, J1.68, J1.70, J1.72, J1.74, J1.76, J1.78, J1.79, J1.8, J1.80, J1.82
- net P1.30: now reaches TP2.1, U4.71 (P1.30)
- net P1.30: now also J1.3
- net P2.10: now reaches TP33.1, U4.134 (P2.10)
- net P2.10: now also J1.65
- net P2.25: now reaches TP23.1, U4.133 (P2.25)
- net P2.25: now also J1.45
- net P0.26: now reaches TP27.1, U4.103 (P0.26)
- net P0.26: now also J1.53
- net P0.18: now reaches TP11.1, U4.32 (P0.18)
- net P0.18: now also J1.21
- net P3.6: now reaches TP14.1, U4.91 (P3.6)
- net P3.6: now also J1.27
- net P1.22: now reaches TP8.1, U4.75 (P1.22)
- net P1.22: now also J1.15
- net P2.0: now reaches TP37.1, U4.120 (P2.0)
- net P2.0: now also J1.73
- net P0.21: now reaches TP9.1, U4.36 (P0.21)
- net P0.21: now also J1.17
- net P1.29: now reaches TP40.1, U4.118 (P1.29)
- net P1.29: now also J1.75
- net P2.5: now reaches TP28.1, U4.125 (P2.5)
- net P2.5: now also J1.55
- net P1.24: now reaches TP20.1, U4.92 (P1.24)
- net P1.24: now also J1.39
- net P0.27: now reaches TP18.1, U4.100 (P0.27)
- net P0.27: now also J1.35
- net P1.26: now reaches TP32.1, U4.115 (P1.26)
- net P1.26: now also J1.63
- net P1.27: now reaches TP41.1, U4.116 (P1.27)
- net P1.27: now also J1.77
- net P1.28: now reaches TP31.1, U4.117 (P1.28)
- net P1.28: now also J1.61
- net P2.1: now reaches TP30.1, U4.121 (P2.1)
- net P2.1: now also J1.59
- net P2.2: now reaches TP36.1, U4.122 (P2.2)
- net P2.2: now also J1.71
- net P2.3: now reaches TP29.1, U4.123 (P2.3)
- net P2.3: now also J1.57
- net P2.4: now reaches TP35.1, U4.124 (P2.4)
- net P2.4: now also J1.69
- net P2.6: now reaches TP26.1, U4.127 (P2.6)
- net P2.6: now also J1.51
- net P2.7: now reaches TP25.1, U4.129 (P2.7)
- net P2.7: now also J1.49
- net P2.8: now reaches TP34.1, U4.130 (P2.8)
- net P2.8: now also J1.67
- net P2.9: now reaches TP24.1, U4.131 (P2.9)
- net P2.9: now also J1.47
- net P0.16: now reaches TP13.1, U4.30 (P0.16)
- net P0.16: now also J1.25
- net P0.17: now reaches TP12.1, U4.31 (P0.17)
- net P0.17: now also J1.23
- net P0.20: now reaches TP10.1, U4.35 (P0.20)
- net P0.20: now also J1.19
- net P1.4: now reaches TP6.1, U4.45 (P1.4)
- net P1.4: now also J1.11
- net P1.8: now reaches TP5.1, U4.46 (P1.8)
- net P1.8: now also J1.9
- net P1.9: now reaches TP4.1, U4.48 (P1.9)
- net P1.9: now also J1.7
- net P1.6: now reaches TP7.1, U4.49 (P1.6)
- net P1.6: now also J1.13
- net P1.23: now reaches TP3.1, U4.70 (P1.23)
- net P1.23: now also J1.5
- net P1.25: now reaches TP1.1, U4.72 (P1.25)
- net P1.25: now also J1.1
- net P3.9: now reaches TP19.1, U4.90 (P3.9)
- net P3.9: now also J1.37
- net P1.31: now reaches TP15.1, U4.93 (P1.31)
- net P1.31: now also J1.29
- net P3.8: now reaches TP21.1, U4.94 (P3.8)
- net P3.8: now also J1.41
- net P3.5: now reaches TP16.1, U4.95 (P3.5)
- net P3.5: now also J1.31
- net P3.7: now reaches TP17.1, U4.96 (P3.7)
- net P3.7: now also J1.33
- net P3.4: now reaches TP22.1, U4.97 (P3.4)
- net P3.4: now also J1.43

Commit message: development backup
Parts:
- renumbered C33 to C1, C21 to C10, C25 to C11, C26 to C12, C27 to C13, C34 to C14, C5 to C15, C38 to C16, C28 to C17, C9 to C18, C29 to C19, C13 to C2, C10 to C20, C4 to C21, C6 to C22, C7 to C23, C30 to C24, C11 to C25, C31 to C26, C1 to C27, C12 to C28, C2 to C29, C17 to C3, C3 to C30, C36 to C31, C35 to C33, C37 to C34, C15 to C35, C16 to C36, C22 to C37, C23 to C38, C19 to C4, C24 to C5, C8 to C6, C14 to C7, C18 to C8, C20 to C9, J2 to J1, J1 to J2, R8 to R4, R9 to R5, R4 to R6, R6 to R7, R5 to R8, R7 to R9, TP38 to TP1, TP6 to TP10, TP7 to TP11, TP8 to TP12, TP9 to TP13, TP10 to TP14, TP11 to TP15, TP12 to TP16, TP13 to TP17, TP14 to TP18, TP15 to TP19, TP42 to TP2, TP16 to TP20, TP17 to TP21, TP18 to TP22, TP19 to TP23, TP20 to TP24, TP21 to TP25, TP22 to TP26, TP23 to TP27, TP24 to TP28, TP25 to TP29, TP39 to TP3, TP26 to TP30, TP27 to TP31, TP28 to TP32, TP29 to TP33, TP30 to TP34, TP31 to TP35, TP32 to TP36, TP33 to TP37, TP34 to TP38, TP35 to TP39, TP43 to TP4, TP36 to TP40, TP37 to TP41, TP40 to TP42, TP41 to TP43, TP1 to TP5, TP2 to TP6, TP3 to TP7, TP4 to TP8, TP5 to TP9, U3 to U1, U5 to U2, U1 to U3, U2 to U5
Connections:
- net 3V3: now also J2.82
- net GND: no longer J2.82

Commit message: test workflow render
Parts:
- added C39: C, Capacitor_SMD:C_0805_2012Metric, symbol Device:C
Changed lines of the file:
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@@
+	)
+	(symbol
+		(lib_id "Device:C")
+		(at 63.5 142.24 0)
+		(unit 1)
+		(exclude_from_sim no)
+		(in_bom yes)
+		(on_board yes)
+		(dnp no)
+		(fields_autoplaced yes)
+		(property "Reference" "C39"
+			(at 67.31 140.9699 0)
+			(effects
+				(font
+					(size 1.27 1.27)
+				)
+				(justify left)
+			)
+		)
+		(property "Value" "C"
+			(at 67.31 143.5099 0)
+			(effects
+				(font
+					(size 1.27 1.27)
+				)
+				(justify left)
+			)
+		)
+		(property "Footprint" "Capacitor_SMD:C_0805_2012Metric"
+			(at 64.4652 146.05 0)
+			(effects
+				(font
+					(size 1.27 1.27)
+				)
+				(hide yes)
+			)
+		)
+		(property "Datasheet" "~"
+			(at 63.5 142.24 0)
+			(effects
+				(font
+					(size 1.27 1.27)
+				)
+				(hide yes)
+			)
+		)
+		(property "Description" "Unpolarized capacitor"
+			(at 63.5 142.24 0)
+			(effects
+				(font
+					(size 1.27 1.27)
+				)
+				(hide yes)
+			)
+		)
+		(pin "1"
+		)
+		(pin "2"
+		)
+		(instances
+			(project ""
+				(path "/95623a5c-6e9d-4c1c-be90-b39230c07c79"
+					(reference "C39")
+					(unit 1)
+				)
+			)
+		)
 	)
 	(symbol

Commit message: test workflow render 2
Parts:
- removed C39: C, Capacitor_SMD:C_0805_2012Metric, symbol Device:C
Changed lines of the file:
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@@
-	)
-	(symbol
-		(lib_id "Device:C")
-		(at 63.5 142.24 0)
-		(unit 1)
-		(exclude_from_sim no)
-		(in_bom yes)
-		(on_board yes)
-		(dnp no)
-		(fields_autoplaced yes)
-		(property "Reference" "C39"
-			(at 67.31 140.9699 0)
-			(effects
-				(font
-					(size 1.27 1.27)
-				)
-				(justify left)
-			)
-		)
-		(property "Value" "C"
-			(at 67.31 143.5099 0)
-			(effects
-				(font
-					(size 1.27 1.27)
-				)
-				(justify left)
-			)
-		)
-		(property "Footprint" "Capacitor_SMD:C_0805_2012Metric"
-			(at 64.4652 146.05 0)
-			(effects
-				(font
-					(size 1.27 1.27)
-				)
-				(hide yes)
-			)
-		)
-		(property "Datasheet" "~"
-			(at 63.5 142.24 0)
-			(effects
-				(font
-					(size 1.27 1.27)
-				)
-				(hide yes)
-			)
-		)
-		(property "Description" "Unpolarized capacitor"
-			(at 63.5 142.24 0)
-			(effects
-				(font
-					(size 1.27 1.27)
-				)
-				(hide yes)
-			)
-		)
-		(pin "1"
-		)
-		(pin "2"
-		)
-		(instances
-			(project ""
-				(path "/95623a5c-6e9d-4c1c-be90-b39230c07c79"
-					(reference "C39")
-					(unit 1)
-				)
-			)
-		)
 	)
 	(symbol

Commit message: development backup
Parts:
- removed MB1: mouse-bite-midle-50mil-200mil, mouse_bite_footprints:mouse-bite-50mil-2138mil, symbol UNITED_MOUSE_BITES_DATA_BASE:mouse-bite-50mil-2138mil
- added J1: CLP-113-02-G-D-BE, connector_footprints:CLP-113-02-G-D-BE, symbol UNITED_CONNECTORS_DATA_BASE:J_CLP-113-02-G-D-BE
- added MB1: mouse-bite-50mil-750mil, mouse_bite_footprints:mouse-bite-50mil-750mil, symbol UNITED_MOUSE_BITES_DATA_BASE:mouse-bite-50mil-750mil
- added MB2: mouse-bite-50mil-1550mil, mouse_bite_footprints:mouse-bite-50mil-1550mil, symbol UNITED_MOUSE_BITES_DATA_BASE:mouse-bite-50mil-1550mil
- added TP1: TestPoint, test_point_footprints:TestPoint_THTPad_Castelated, symbol UNITED_TEST_POINTS:TestPoint_Castelated
- J2: value CLP-150-02-G-D-BE -> CLP-129-02-G-D-BE; footprint connector_footprints:CLP-141-02-G-D-BE -> connector_footprints:CLP-129-02-G-D-BE; symbol UNITED_CONNECTORS_DATA_BASE:J_CLP-141-02-G-D-BE -> UNITED_CONNECTORS_DATA_BASE:J_CLP-129-02-G-D-BE; MPN CLP-141-02-G-D-BE -> CLP-129-02-G-D-BE; Pin Count 41 -> 29; Symbol Name J_CLP-141-02-G-D-BE -> J_CLP-129-02-G-D-BE; Trustedparts Search https://www.trustedparts.com/en/search/CLP-141-02-G-D-BE -> https://www.trustedparts.com/en/search/CLP-129-02-G-D-BE
- renumbered C30 to C1, C25 to C10, C20 to C11, C18 to C12, C7 to C13, C2 to C14, C35 to C15, C36 to C16, C8 to C17, C3 to C18, C9 to C19, C29 to C2, C4 to C20, C10 to C21, C38 to C22, C37 to C23, C11 to C24, C5 to C25, C12 to C26, C13 to C27, C32 to C28, C26 to C29, C27 to C3, C24 to C30, C19 to C31, C17 to C32, C1 to C33, C14 to C34, C16 to C35, C33 to C36, C34 to C37, C31 to C38, C21 to C4, C15 to C5, C22 to C6, C23 to C7, C6 to C8, C28 to C9, D2 to D1, D1 to D2, J1 to J3, Q2 to Q1, Q1 to Q2, R8 to R4, R6 to R5, R9 to R6, R5 to R8, R4 to R9, TP8 to TP10, TP7 to TP11, TP6 to TP12, TP5 to TP13, TP17 to TP14, TP18 to TP15, TP19 to TP16, TP20 to TP17, TP21 to TP18, TP22 to TP19, TP16 to TP2, TP23 to TP20, TP24 to TP21, TP25 to TP22, TP26 to TP23, TP27 to TP24, TP28 to TP25, TP29 to TP26, TP30 to TP27, TP31 to TP28, TP32 to TP29, TP15 to TP3, TP33 to TP30, TP34 to TP31, TP35 to TP32, TP36 to TP33, TP37 to TP34, TP38 to TP35, TP39 to TP36, TP40 to TP37, TP41 to TP38, TP3 to TP39, TP14 to TP4, TP1 to TP40, TP42 to TP41, TP43 to TP42, TP4 to TP43, TP2 to TP44, TP44 to TP45, TP45 to TP46, TP13 to TP5, TP12 to TP6, TP11 to TP7, TP10 to TP8, U3 to U1, U5 to U2, U1 to U3, U2 to U5
Connections:
- net 3V3: now also J2.1, J2.2; no longer J2.81, J2.82
- net GND: now also J2.11, J2.13, J2.15, J2.17, J2.19, J2.21, J2.23, J2.25, J2.27, J2.29, J2.3, J2.31, J2.33, J2.35, J2.37, J2.39, J2.41, J2.43, J2.45, J2.47, J2.49, J2.5, J2.51, J2.53, J2.55, J2.57, J2.7, J2.9, J1.1, J1.11, J1.13, J1.15, J1.17, J1.19, J1.2, J1.21, J1.23, J1.25, J1.3, J1.5, J1.7, J1.9, TP1.1; no longer J2.10, J2.12, J2.14, J2.16, J2.18, J2.2, J2.20, J2.22, J2.24, J2.26, J2.28, J2.30, J2.32, J2.34, J2.36, J2.38, J2.40, J2.42, J2.44, J2.46, J2.48, J2.50, J2.52, J2.54, J2.56, J2.58, J2.6, J2.60, J2.62, J2.64, J2.66, J2.68, J2.70, J2.72, J2.74, J2.76, J2.78, J2.79, J2.8, J2.80
- net P0.16: now also J2.58; no longer J2.25
- net P0.17: now also J1.4; no longer J2.23
- net P0.18: now also J1.6; no longer J2.21
- net P0.20: now also J1.8; no longer J2.19
- net P0.21: now also J1.10; no longer J2.17
- net P0.26: now also J2.30; no longer J2.53
- net P0.27: now also J2.48; no longer J2.35
- net P1.22: now also J1.12; no longer J2.15
- net P1.23: now also J1.22; no longer J2.5
- net P1.24: now also J2.44; no longer J2.39
- net P1.25: now also J1.26; no longer J2.1
- net P1.26: now also J2.20; no longer J2.63
- net P1.27: now also J2.6; no longer J2.77
- net P1.28: now also J2.22; no longer J2.61
- net P1.29: now also J2.8; no longer J2.75
- net P1.30: now also J1.24; no longer J2.3
- net P1.31: now also J2.54; no longer J2.29
- net P1.4: now also J1.16; no longer J2.11
- net P1.6: now also J1.14; no longer J2.13
- net P1.8: now also J1.18; no longer J2.9
- net P1.9: now also J1.20; no longer J2.7
- net P2.0: now also J2.10; no longer J2.73
- net P2.1: now also J2.24; no longer J2.59
- net P2.10: now also J2.18; no longer J2.65
- net P2.2: now also J2.12; no longer J2.71
- net P2.25: now also J2.38; no longer J2.45
- net P2.3: now also J2.26; no longer J2.57
- net P2.4: now also J2.14; no longer J2.69
- net P2.5: now also J2.28; no longer J2.55
- net P2.6: now also J2.32; no longer J2.51
- net P2.7: now also J2.34; no longer J2.49
- net P2.8: now also J2.16; no longer J2.67
- net P2.9: now also J2.36; no longer J2.47
- net P3.4: now also J2.40; no longer J2.43
- net P3.5: now also J2.52; no longer J2.31
- net P3.6: now also J2.56; no longer J2.27
- net P3.7: now also J2.50; no longer J2.33
- net P3.8: now also J2.42; no longer J2.41
- net P3.9: now also J2.46; no longer J2.37
Other:
- moved on the sheet: C36, C37, C38, R4, R5, R6, R7, TP39, TP40, TP43, TP44, TP45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

Commit message: development backup
Parts:
- added C39: 100 nF, capacitor_footprints:C_0402_1005Metric, symbol UNITED_CAPACITORS_DATA_BASE:C_GCM155R71H104KE02D
- added R10: 10k, resistor_footprints:R_0402_1005Metric, symbol UNITED_RESISTORS_DATA_BASE:R_ERJ-2RKF1002X
- added R11: 10 Ω, resistor_footprints:R_0402_1005Metric, symbol UNITED_RESISTORS_DATA_BASE:R_ERJ-2RKF10R0X
- added S1: TS21-34-035-BK-160-SMT-TR, tactile_switches_footprints:TS21, symbol UNITED_TACTILE_SWITCHES_DATA_BASE:S_TS21-34-035-BK-160-SMT-TR
Connections:
- net 3V3: now also R10.1
- net GND: now also R11.2, S1.3, S1.4
- net RSTN: now also C39.1, R10.2, S1.1, S1.2
- new net: C39.2, R11.1
Other:
- moved on the sheet: C35, J3
