File: minimal_max32650/minimal_max32650.kicad_pcb (KiCad board)
At the start: 4 copper layers, 52.7 x 46.4 mm, 108 parts, among them J1 CLP-113-02-G-D-BE, J2 CLP-129-02-G-D-BE, J3 FTSH-105-01-L-DV-K, Q1 50 V, Q2 50 V, U1 ADT75BRMZ, U2 S80KS5122GABHM020, U3 MX25U6432FZNI02, U4 MAX32650GCE+, U5 MAXQ1065GTC+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

Commit message: development backup
Parts:
- added REF**: OSHW-Logo_5.7x6mm_SilkScreen, Symbol:OSHW-Logo_5.7x6mm_SilkScreen, F.Cu at (177.7, 103.5)
- added REF**: KiCad-Logo2_5mm_SilkScreen, Symbol:KiCad-Logo2_5mm_SilkScreen, F.Cu at (146.7, 87.4)

Commit message: development backup
Parts:
- removed REF**: OSHW-Logo_5.7x6mm_SilkScreen, Symbol:OSHW-Logo_5.7x6mm_SilkScreen
- removed REF**: KiCad-Logo2_5mm_SilkScreen, Symbol:KiCad-Logo2_5mm_SilkScreen
- added C39: 100 nF, capacitor_footprints:C_0402_1005Metric, F.Cu at (189.7, 91.2)
- added R10: 10k, resistor_footprints:R_0402_1005Metric, F.Cu at (179.5, 96.7)
- added R11: 10 Ω, resistor_footprints:R_0402_1005Metric, F.Cu at (189.6, 92.3)
- added S1: TS21-34-035-BK-160-SMT-TR, tactile_switches_footprints:TS21, F.Cu at (186.0, 92.2)
- moved Q1 5.43 mm to (189.9, 76.4)
- moved D1 5.43 mm to (189.5, 78.7)
- moved R8 5.30 mm to (189.5, 79.9), turned to 180 degrees
- moved C35 4.26 mm to (190.5, 84.7), turned to -90 degrees
- moved J3 2.79 mm to (186.3, 86.8)
- moved R9 1.79 mm to (185.9, 79.9), turned to 180 degrees
- moved D2 1.22 mm to (185.8, 78.7)
- moved Q2 1.22 mm to (186.3, 76.4)
Routing:
- net /RSTN: track 10.8 -> 19.8 mm
- net /LED2: track 13.5 -> 19.1 mm
- net /3V3: track 35.7 -> 39.4 mm, vias 21 -> 22
- net /UART0_TX: track 10.9 -> 8.30 mm
- net /TCK: track 18.1 -> 20.6 mm
- net /LED1: track 17.6 -> 15.5 mm
- net /UART0_RX: track 9.49 -> 7.92 mm
- net /TMS: track 17.9 -> 19.3 mm
- net Net-(C39-Pad2): track 0.00 -> 1.18 mm
- net GND: vias 66 -> 69

Commit message: development backup
Parts:
- moved C35 0.39 mm to (190.5, 84.3)
- moved J3 0.39 mm to (186.3, 86.4)
- moved C39 0.09 mm to (189.7, 91.1)
- moved S1 0.09 mm to (186.0, 92.1)
- moved R11 0.09 mm to (189.6, 92.2)
Routing:
- net /RSTN: track 19.8 -> 20.7 mm
- net /TMS: track 19.3 -> 19.9 mm
